File: board/display.kicad_sch (KiCad schematic)
At the start: 58 parts

Commit message: Lots of silly train things
Parts:
- C11: footprint (none) -> Capacitor_SMD:C_0805_2012Metric
- R12: footprint (none) -> Resistor_SMD:R_0805_2012Metric
Other:
- note added: "Nottingham"
Changed lines of the file:
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@@
 		)
 	)
-	(text "Derby"
+	(text "Nottingham"
 		(exclude_from_sim no)
-		(at 16.51 144.272 0)
+		(at 22.352 144.272 0)
 		(effects
 			(font
@@
 			)
 		)
-		(property "Footprint" ""
+		(property "Footprint" "Resistor_SMD:R_0805_2012Metric"
 			(at 19.05 28.448 90)
 			(effects
@@
 			)
 		)
-		(property "Footprint" ""
+		(property "Footprint" "Capacitor_SMD:C_0805_2012Metric"
 			(at 268.9352 26.67 0)
 			(effects

Commit message: Lay out some stations
Connections:
- net GND: now also D10.3 (VSS), D11.3 (VSS), D12.3 (VSS), D13.3 (VSS), D14.3 (VSS), D15.3 (VSS), D16.3 (VSS), D6.3 (VSS), D7.3 (VSS), D8.3 (VSS), D9.3 (VSS)
Changed lines of the file:
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@@
 	)
 	(junction
+		(at 246.38 34.29)
+		(diameter 0)
+		(color 0 0 0 0)
+	)
+	(junction
 		(at 200.66 95.25)
 		(diameter 0)
@@
 	(wire
 		(pts
+			(xy 24.13 43.18) (xy 24.13 46.99)
+		)
+		(stroke
+			(width 0)
+			(type default)
+		)
+	)
+	(wire
+		(pts
 			(xy 245.11 163.83) (xy 267.97 163.83)
 		)
@@
 	(wire
 		(pts
-			(xy 254 26.67) (xy 254 35.56)
+			(xy 22.86 43.18) (xy 24.13 43.18)
 		)
 		(stroke
@@
 	(wire
 		(pts
-			(xy 254 35.56) (xy 24.13 35.56)
+			(xy 254 40.64) (xy 22.86 40.64)
 		)
 		(stroke
@@
 	(wire
 		(pts
-			(xy 24.13 35.56) (xy 24.13 46.99)
+			(xy 22.86 40.64) (xy 22.86 43.18)
 		)
 		(stroke
@@
 	(wire
 		(pts
+			(xy 254 26.67) (xy 254 40.64)
+		)
+		(stroke
+			(width 0)
+			(type default)
+		)
+	)
+	(wire
+		(pts
 			(xy 125.73 58.42) (xy 125.73 46.99)
 		)
@@
 					(unit 1)
 				)
+			)
+		)
+	)
+	(symbol
+		(lib_id "power:GND")
+		(at 246.38 34.29 0)
+		(unit 1)
+		(exclude_from_sim no)
+		(in_bom yes)
+		(on_board yes)
+		(dnp no)
+		(fields_autoplaced yes)
+		(property "Reference" "#PWR075"
+			(at 246.38 40.64 0)
+			(effects
+				(font
+					(size 1.27 1.27)
+				)
+				(hide yes)
+			)
+		)
+		(property "Value" "GND"
+			(at 246.38 39.37 0)
+			(effects
+				(font
+					(size 1.27 1.27)
+				)
+			)
+		)
+		(property "Footprint" ""
+			(at 246.38 34.29 0)
+			(effects
+				(font
+					(size 1.27 1.27)
+				)
+				(hide yes)
+			)
+		)
+		(property "Datasheet" ""
+			(at 246.38 34.29 0)
+			(effects
+				(font
+					(size 1.27 1.27)
+				)
+				(hide yes)
+			)
+		)
+		(property "Description" "Power symbol creates a global label with name \"GND\" , ground"
+			(at 246.38 34.29 0)
+			(effects
+				(font
+					(size 1.27 1.27)
+				)
+				(hide yes)
+			)
+		)
+		(pin "1"
+		)
+		(instances
+			(project ""
+				(path "/380d0889-29f1-4d98-b1bb-ce6ede3c8d67/1f31e997-0b33-46b7-9567-f7802b85367a"
+					(reference "#PWR075")
+					(unit 1)
+				)
