File: board/board.kicad_pcb (KiCad board)
At the start: 2 copper layers, 141 parts, among them IC1 HUSB238, J1 USB_C_Receptacle_USB2.0_14P, J2 USB_C_Receptacle_USB2.0_14P, Q1 IRLML6402TRPBF, SW1 SW_Push, SW2 SW_Push, U1 SED5120, U2 TXB0106PW, U3 ESP32-S3-WROOM-1

Commit message: Micrcontroller, but wired up
Parts:
- added C13: 0.1uF, Capacitor_SMD:C_0805_2012Metric, F.Cu at (52.0, 66.2)
- added RST: SW_Push, LCSC:SW-SMD_4P-L4.2-W3.3-P2.15-LS5.1, F.Cu at (51.8, 70.3)
- moved BOOT 172.9 mm to (63.7, 36.4), turned to -90 degrees
- moved J2 162.6 mm to (62.0, 118.2)
- moved USER 159.9 mm to (58.5, 61.6)
- moved U2 156.2 mm to (54.3, 31.9), turned to 180 degrees
- moved J1 146.5 mm to (51.4, 118.2)
- moved GENERAL 144.5 mm to (53.9, 80.6)
- moved SERVER 143.3 mm to (53.9, 82.7)
- moved U3 142.3 mm to (52.3, 49.4), turned to 90 degrees
- moved WIFI 142.2 mm to (53.9, 84.7)
- moved R1 133.3 mm to (52.0, 102.9)
- moved R3 131.8 mm to (52.7, 105.7), turned to 90 degrees
- moved R2 131.1 mm to (48.2, 106.5), turned to -90 degrees
- moved IC1 125.7 mm to (51.4, 109.5), turned to 90 degrees
- moved R4 123.2 mm to (57.3, 88.8), turned to 180 degrees
- moved C6 122.4 mm to (59.2, 32.1), turned to 90 degrees
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- renumbered D2 to 3V3, D1 to 5V, SW1 to BOOT, D5 to GENERAL, D4 to SERVER, SW2 to USER, D3 to WIFI
Connections:
- net Net-(U3-EN) renamed /Micrcontroller/EN
- U3 pad 15: /Micrcontroller/GENERAL_STATUS_LED -> /Micrcontroller/NEOPIXELS
- U3 pad 38: /Micrcontroller/SERVER_STATUS_LED -> unconnected-(U3-IO2-Pad38)
- U3 pad 39: /Micrcontroller/WIFI_STATUS_LED -> unconnected-(U3-IO1-Pad39)
- U3 pad 5: /Micrcontroller/NEOPIXELS -> /Micrcontroller/GENERAL_STATUS_LED
- U3 pad 6: unconnected-(U3-IO6-Pad6) -> /Micrcontroller/SERVER_STATUS_LED
- U3 pad 7: unconnected-(U3-IO7-Pad7) -> /Micrcontroller/WIFI_STATUS_LED
Routing:
- net +3V3: track 0.00 -> 91.5 mm, vias 0 -> 2
- net /Micrcontroller/USB_D-: track 0.00 -> 60.8 mm
- net /Micrcontroller/USB_D+: track 0.00 -> 59.6 mm
- net GND: track 0.00 -> 50.7 mm, vias 0 -> 14
- net /Micrcontroller/NEOPIXELS: track 0.00 -> 33.3 mm
- net /Micrcontroller/WIFI_STATUS_LED: track 0.00 -> 29.0 mm
- net /Micrcontroller/SERVER_STATUS_LED: track 0.00 -> 27.2 mm
- net /Micrcontroller/GENERAL_STATUS_LED: track 0.00 -> 25.0 mm
- net Net-(Q1-Bulk): track 0.00 -> 25.0 mm
- net +5V: track 0.00 -> 15.8 mm, vias 0 -> 2
- net /Micrcontroller/EN: track 0.00 -> 14.0 mm
- net /Micrcontroller/USER_BUTTON: track 0.00 -> 12.3 mm, vias 0 -> 2
- net Net-(IC1-D-): track 0.00 -> 8.84 mm, vias 0 -> 2
- net Net-(Q1-G): track 0.00 -> 8.07 mm
- net NEOPIXELS_SHIFTED: track 0.00 -> 7.72 mm
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- added copper zone on F.Cu, net +5V
- added copper zone on B.Cu, net GND
Other:
- board outline added: 100 x 100 mm

Commit message: Lay out some stations
Parts:
- moved D68 304.0 mm to (253.4, 63.9)
- moved D67 302.3 mm to (253.4, 69.5)
- moved D66 301.1 mm to (253.4, 75.2)
- moved D41 295.8 mm to (223.7, 69.4)
- moved D42 294.6 mm to (223.8, 63.8)
- moved D39 290.7 mm to (216.7, 69.4)
- moved D40 288.9 mm to (216.7, 63.8)
- moved D37 287.8 mm to (209.6, 69.4)
- moved D65 287.7 mm to (239.5, 63.9)
- moved D64 286.8 mm to (239.5, 69.5)
- moved D62 286.5 mm to (239.5, 80.8)
- moved D63 286.4 mm to (239.5, 75.1)
- moved D38 284.0 mm to (209.6, 63.8)
- moved D35 281.5 mm to (202.6, 69.4)
- moved D36 280.7 mm to (202.6, 63.8)
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- renumbered BOOT to SW1, USER to SW2, RST to SW3
Connections:
- D10 pad 3: Net-(D10-VSS) -> GND
- D11 pad 3: Net-(D10-VSS) -> GND
- D12 pad 3: Net-(D10-VSS) -> GND
- D13 pad 3: Net-(D10-VSS) -> GND
- D14 pad 3: Net-(D10-VSS) -> GND
- D15 pad 3: Net-(D10-VSS) -> GND
- D16 pad 3: Net-(D10-VSS) -> GND
- D6 pad 3: Net-(D10-VSS) -> GND
- D65 pad 2: GND -> Net-(D65-DOUT)
- D66 pad 4: GND -> Net-(D65-DOUT)
- D7 pad 3: Net-(D10-VSS) -> GND
- D8 pad 3: Net-(D10-VSS) -> GND
- D9 pad 3: Net-(D10-VSS) -> GND
Routing:
- net Net-(D42-DOUT): track 0.00 -> 93.0 mm
- net GND: track 50.7 -> 129.4 mm, vias 14 -> 70
- net NEOPIXELS_SHIFTED_PG2: track 0.00 -> 61.8 mm
- net Net-(D26-DOUT): track 0.00 -> 36.8 mm
- net Net-(D65-DOUT): track 0.00 -> 35.5 mm
- net Net-(D44-DOUT): track 0.00 -> 34.5 mm
- net Net-(D19-DOUT): track 0.00 -> 31.1 mm
- net Net-(D28-DOUT): track 0.00 -> 30.1 mm
- net Net-(D23-DOUT): track 0.00 -> 29.1 mm
- net Net-(D21-DOUT): track 0.00 -> 27.5 mm
- net Net-(D32-DOUT): track 0.00 -> 25.5 mm
- net Net-(D30-DOUT): track 0.00 -> 25.5 mm
- net Net-(D34-DOUT): track 0.00 -> 25.5 mm
- net Net-(D36-DOUT): track 0.00 -> 25.4 mm
- net Net-(D38-DOUT): track 0.00 -> 25.4 mm
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Other:
- board size 100 x 100 mm -> 239.4 x 100 mm
- board text added: "ALF"
- board text added: "ALFRETON"
- board text added: "BELPER"
- board text added: "BLP"
- board text added: "CHESTERFIELD"
- board text added: "CHF"
- board text added: "DBY"
- board text added: "DERBY"
- board text added: "DRO"
- board text added: "DRONFIELD"
- board text added: "EAST MIDLANDS PARKWAY"
- board text added: "EMD"
- board text added: "LBO"
- board text added: "LOUGHBOROUGH"
- board text added: "NOT"
- board text added: "NOTTINGHAM"
- board text added: "Plat 1"
- board text added: "Plat 1a"
- board text added: "Plat 7"
- board text added: "Plat 8a"
- board text added: "SHEFFIELD"
- board text added: "SHF"

Commit message: Finishing touches on the PCB
Parts:
- added H1: MountingHole, MountingHole:MountingHole_2.2mm_M2, F.Cu at (48.5, 25.4)
- added H2: MountingHole, MountingHole:MountingHole_2.2mm_M2, F.Cu at (165.2, 25.4)
- added H3: MountingHole, MountingHole:MountingHole_2.2mm_M2, F.Cu at (281.9, 25.4)
- added H4: MountingHole, MountingHole:MountingHole_2.2mm_M2, F.Cu at (281.9, 119.5)
- added H5: MountingHole, MountingHole:MountingHole_2.2mm_M2, F.Cu at (165.2, 119.5)
- added H6: MountingHole, MountingHole:MountingHole_2.2mm_M2, F.Cu at (72.7, 119.5)
- moved D93 287.1 mm to (259.4, 63.8)
- moved D92 285.0 mm to (259.4, 69.4)
- moved D101 285.0 mm to (266.5, 69.4)
- moved D108 284.6 mm to (266.4, 30.0)
- moved D100 283.2 mm to (266.5, 75.0)
- moved D99 281.9 mm to (266.5, 80.6)
- moved D107 281.3 mm to (266.5, 35.6)
- moved D96 281.2 mm to (266.5, 97.5)
- moved D98 281.1 mm to (266.5, 86.2)
- moved D97 280.9 mm to (266.5, 91.9)
- moved D106 278.6 mm to (266.5, 41.2)
- moved D83 278.2 mm to (245.3, 69.4)
- moved D91 277.2 mm to (252.4, 69.4)
- moved D90 277.0 mm to (252.4, 63.8)
- moved D89 276.9 mm to (252.4, 58.1)
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Connections:
- D70 pad 2: unconnected-(D70-DOUT-Pad2) -> Net-(D70-DOUT)
- D71 pad 4: unconnected-(D71-DIN-Pad4) -> Net-(D70-DOUT)
- D76 pad 2: unconnected-(D76-DOUT-Pad2) -> Net-(D76-DOUT)
- D77 pad 4: unconnected-(D77-DIN-Pad4) -> Net-(D76-DOUT)
- D81 pad 2: unconnected-(D81-DOUT-Pad2) -> Net-(D81-DOUT)
- D82 pad 4: unconnected-(D82-DIN-Pad4) -> Net-(D81-DOUT)
- D86 pad 2: unconnected-(D86-DOUT-Pad2) -> Net-(D86-DOUT)
- D87 pad 4: unconnected-(D87-DIN-Pad4) -> Net-(D86-DOUT)
- D91 pad 2: unconnected-(D91-DOUT-Pad2) -> Net-(D91-DOUT)
- D92 pad 4: unconnected-(D92-DIN-Pad4) -> Net-(D91-DOUT)
Routing:
- net GND: track 129.4 -> 280.1 mm, vias 70 -> 123
- net Net-(D95-DOUT): track 0.00 -> 64.8 mm
- net NEOPIXELS_SHIFTED: track 7.72 -> 61.0 mm
- net Net-(D72-DOUT): track 0.00 -> 37.6 mm
- net Net-(D78-DOUT): track 0.00 -> 36.7 mm
- net Net-(D68-DOUT): track 0.00 -> 31.1 mm
- net Net-(D74-DOUT): track 0.00 -> 25.6 mm
- net Net-(D81-DOUT): track 0.00 -> 24.4 mm
- net Net-(D86-DOUT): track 0.00 -> 22.6 mm
- net Net-(D83-DOUT): track 0.00 -> 18.3 mm
- net Net-(D42-DOUT): track 93.0 -> 78.2 mm
- net Net-(D91-DOUT): track 0.00 -> 13.9 mm
- net Net-(D59-DOUT): track 0.00 -> 13.3 mm
- net Net-(D82-DOUT): track 0.00 -> 13.3 mm
- net Net-(D49-DOUT): track 0.00 -> 13.3 mm
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- added copper zone on In1.Cu, net +5V
Other:
- copper layers 2 -> 4
- board text added: "BDM"
- board text added: "CHD"
- board text added: "KET"
- board text added: "LEI"
- board text added: "LUT"
- board text added: "MHR"
- board text added: "Plat 5"
- board text added: "Plat 7a"
- board text added: "SAC"
- board text added: "STP"
- board text added: "WEL"
- board text removed: "ALFRETON"
- board text removed: "BELPER"
- board text removed: "CHESTERFIELD"
- board text removed: "CHF"
- board text removed: "DERBY"
- board text removed: "DRONFIELD"
- board text removed: "EAST MIDLANDS PARKWAY"
- board text removed: "LOUGHBOROUGH"
- board text removed: "NOTTINGHAM"
- board text removed: "SHEFFIELD"
