File: board/display2.kicad_sch (KiCad schematic)
At the start: 48 parts

Commit message: Lots of silly train things
Parts:
- C12: footprint (none) -> Capacitor_SMD:C_0805_2012Metric
Other:
- note added: "Luton"
Changed lines of the file:
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@@
 		)
 	)
-	(text "Bedford"
+	(text "Luton"
 		(exclude_from_sim no)
-		(at 136.652 70.612 0)
+		(at 134.62 70.612 0)
 		(effects
 			(font
@@
 			)
 		)
-		(property "Footprint" ""
+		(property "Footprint" "Capacitor_SMD:C_0805_2012Metric"
 			(at 110.1852 26.67 0)
 			(effects

Commit message: Lay out some stations
Connections:
- net GND: no longer D65.2 (DOUT), D66.4 (DIN)
- new net: D65.2 (DOUT), D66.4 (DIN)
Changed lines of the file:
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@@
-	)
-	(junction
-		(at 109.22 26.67)
-		(diameter 0)
-		(color 0 0 0 0)
 	)
 	(junction
@@
 	(wire
 		(pts
+			(xy 97.79 34.29) (xy 97.79 26.67)
+		)
+		(stroke
+			(width 0)
+			(type default)
+		)
+	)
+	(wire
+		(pts
 			(xy 104.14 46.99) (xy 125.73 46.99)
 		)
@@
 	(wire
 		(pts
-			(xy 97.79 26.67) (xy 109.22 26.67)
+			(xy 97.79 34.29) (xy 125.73 34.29)
 		)
 		(stroke
@@
 	(wire
 		(pts
+			(xy 125.73 34.29) (xy 125.73 26.67)
+		)
+		(stroke
+			(width 0)
+			(type default)
+		)
+	)
+	(wire
+		(pts
 			(xy 254 138.43) (xy 261.62 138.43)
 		)
@@
 		)
 		(stroke
-			(width 0)
-			(type default)
-		)
-	)
-	(wire
-		(pts
-			(xy 109.22 26.67) (xy 125.73 26.67)
-		)
-		(stroke

Commit message: Finishing touches on the PCB
Connections:
- net at D76.2 (DOUT): now also D77.4 (DIN)
- net at D70.2 (DOUT): now also D71.4 (DIN)
- net at D82.4 (DIN): now also D81.2 (DOUT)
- net at D87.4 (DIN): now also D86.2 (DOUT)
- net at D91.2 (DOUT): now also D92.4 (DIN)
Changed lines of the file:
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@@
+	(wire
+		(pts
+			(xy 16.51 96.52) (xy 16.51 110.49)
+		)
+		(stroke
+			(width 0)
+			(type default)
+		)
+	)
 	(wire
 		(pts
@@
 	(wire
 		(pts
+			(xy 236.22 96.52) (xy 16.51 96.52)
+		)
+		(stroke
+			(width 0)
+			(type default)
+		)
+	)
+	(wire
+		(pts
 			(xy 113.03 146.05) (xy 91.44 146.05)
 		)
@@
 	(wire
 		(pts
+			(xy 236.22 26.67) (xy 242.57 26.67)
+		)
+		(stroke
+			(width 0)
+			(type default)
+		)
+	)
+	(wire
+		(pts
 			(xy 179.07 26.67) (xy 185.42 26.67)
 		)
@@
 	(wire
 		(pts
+			(xy 111.76 54.61) (xy 118.11 54.61)
+		)
+		(stroke
+			(width 0)
+			(type default)
+		)
+	)
+	(wire
+		(pts
 			(xy 207.01 90.17) (xy 228.6 90.17)
 		)
@@
 	(wire
 		(pts
+			(xy 223.52 54.61) (xy 223.52 66.04)
+		)
+		(stroke
+			(width 0)
+			(type default)
+		)
+	)
+	(wire
+		(pts
 			(xy 104.14 46.99) (xy 125.73 46.99)
 		)
@@
 	(wire
 		(pts
+			(xy 119.38 82.55) (xy 133.35 82.55)
+		)
+		(stroke
+			(width 0)
+			(type default)
+		)
+	)
+	(wire
+		(pts
 			(xy 68.58 146.05) (xy 46.99 146.05)
 		)
@@
 	(wire
 		(pts
-			(xy 8.89 110.49) (xy 16.51 110.49)
-		)
-		(stroke
-			(width 0)
-			(type default)
-		)
-	)
-	(wire
-		(pts
 			(xy 16.51 41.91) (xy 16.51 54.61)
 		)
@@
 	(wire
 		(pts
+			(xy 236.22 82.55) (xy 236.22 96.52)
+		)
+		(stroke
+			(width 0)
+			(type default)
+		)
+	)
+	(wire
+		(pts
 			(xy 68.58 130.81) (xy 91.44 130.81)
 		)
@@
 	(wire
 		(pts
+			(xy 223.52 66.04) (xy 16.51 66.04)
+		)
+		(stroke
+			(width 0)
+			(type default)
+		)
+	)
+	(wire
+		(pts
 			(xy 185.42 74.93) (xy 207.01 74.93)
 		)
@@
 		)
 		(stroke
+			(width 0)
+			(type default)
+		)
+	)
+	(wire
+		(pts
+			(xy 16.51 66.04) (xy 16.51 82.55)
+		)
+		(stroke
